File: shcV1.sch (EAGLE design)
At the start: 19 parts, among them IC1 LM317T, IC2 LM317T, IC3 LM317T, IC4 LM317T

Commit message: Add comment in shc
Other:
- note added: "+Battery"
- note added: "+Vin"
- note added: "Parallel 4 LM317T Iout = 1.5Ax4 = 6A max"
- note added: "Trim for Vout = 13.8V"
Changed lines of the file:
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@@
 <sheet>
 <plain>
+<text x="-40.64" y="40.64" size="1.778" layer="91">+Vin</text>
+<text x="124.46" y="33.02" size="1.778" layer="91">+Battery</text>
+<text x="25.4" y="-10.16" size="1.778" layer="91">Trim for Vout = 13.8V</text>
+<text x="66.04" y="68.58" size="1.778" layer="91">Parallel 4 LM317T  Iout = 1.5Ax4 = 6A max</text>
 </plain>
 <instances>
